File: PCB/PCB.kicad_pcb (KiCad board)
At the start: 2 copper layers, 211 parts, among them J1 Conn_01x04, J2 USB_C_Receptacle_USB2.0_16P, J3 Conn_01x05, SW1 MX_SW_HS, SW10 MX_SW_HS, SW11 MX_SW_HS, SW12 MX_SW_HS, SW13 MX_SW_HS, SW15 MX_SW_HS, SW16 MX_SW_HS, SW17 MX_SW_HS, SW18 MX_SW_HS, SW19 MX_SW_HS, SW2 MX_SW_HS, SW20 MX_SW_HS, SW21 MX_SW_HS, SW22 MX_SW_HS, SW23 MX_SW_HS, SW24 MX_SW_HS, SW25 MX_SW_HS, SW26 MX_SW_HS, SW27 MX_SW_HS, SW28 MX_SW_HS, SW29 MX_SW_HS, SW3 MX_SW_HS, SW30 MX_SW_HS, SW31 MX_SW_HS, SW32 MX_SW_HS, SW33 MX_SW_HS, SW34 MX_SW_HS, SW35 MX_SW_HS, SW36 MX_SW_HS, SW37 MX_SW_HS, SW38 MX_SW_HS, SW39 MX_SW_HS, SW4 MX_SW_HS, SW40 MX_SW_HS, SW41 MX_SW_HS, SW42 MX_SW_HS, SW43 MX_SW_HS, SW44 MX_SW_HS, SW45 MX_SW_HS, SW46 MX_SW_HS, SW47 MX_SW_HS, SW48 MX_SW_HS, SW49 MX_SW_HS, SW5 MX_SW_HS, SW50 MX_SW_HS, SW51 MX_SW_HS, SW52 MX_SW_HS, SW53 MX_SW_HS, SW54 MX_SW_HS, SW55 MX_SW_HS, SW56 MX_SW_HS, SW57 MX_SW_HS, SW58 MX_SW_HS, SW59 MX_SW_HS, SW6 MX_SW_HS, SW60 MX_SW_HS, SW61 MX_SW_HS, SW62 MX_SW_HS, SW63 MX_SW_HS, SW64 MX_SW_HS, SW65 MX_SW_HS, SW66 MX_SW_HS, SW67 MX_SW_HS, SW68 MX_SW_HS, SW69 MX_SW_HS, SW7 MX_SW_HS, SW70 MX_SW_HS, SW71 MX_SW_HS, SW72 MX_SW_HS, SW73 MX_SW_HS, SW74 MX_SW_HS, SW75 MX_SW_HS, SW76 MX_SW_HS, SW77 MX_SW_HS, SW78 MX_SW_HS, SW79 MX_SW_HS, SW8 MX_SW_HS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

Commit message: idk update
Parts:
- added C11: 100n, Capacitor_SMD:C_0402_1005Metric, B.Cu at (131.8, 132.3)
- added C12: 100n, Capacitor_SMD:C_0402_1005Metric, B.Cu at (134.7, 132.3)
- added C13: 100n, Capacitor_SMD:C_0402_1005Metric, B.Cu at (135.1, 144.0)
- added C5: 100n, Capacitor_SMD:C_0402_1005Metric, B.Cu at (135.7, 132.3)
- BOOT1, C1, C2, C3, C4, D1, D10, D11, D12, D13, D2, D3, D4, D5, D6, D7, D8, D9, F1, J1, J2, J3, R1, R2, R3, R4, R5, R6, R7, R8, R9, RST1, S1, S2, S3, SW1, SW10, SW11, SW12, SW13, SW2, SW3, SW4, SW5, SW6, SW7, SW8, SW9, U1, U2, U3, U4, Y1: moved to B.Cu
- C10: renamed from C9; moved to B.Cu
- C14: renamed from C10; moved to B.Cu
- C15: renamed from C11; moved to B.Cu
- C16: renamed from C12; moved to B.Cu
- C6: renamed from C5; moved to B.Cu
- C7: renamed from C6; moved to B.Cu
- C8: renamed from C7; moved to B.Cu
- C9: renamed from C8; moved to B.Cu
- D14: renamed from D15; moved to B.Cu
- D15: renamed from D16; moved to B.Cu
- D16: renamed from D17; moved to B.Cu
- D17: renamed from D18; moved to B.Cu
- D18: renamed from D19; moved to B.Cu
- D19: renamed from D20; moved to B.Cu
- D20: renamed from D21; moved to B.Cu
- D21: renamed from D22; moved to B.Cu
- D22: renamed from D23; moved to B.Cu
- D23: renamed from D24; moved to B.Cu
- D24: renamed from D25; moved to B.Cu
- D25: renamed from D26; moved to B.Cu
- D26: renamed from D27; moved to B.Cu
- D27: renamed from D28; moved to B.Cu
- D28: renamed from D29; moved to B.Cu
- D29: renamed from D30; moved to B.Cu
- D30: renamed from D31; moved to B.Cu
- D31: renamed from D32; moved to B.Cu
- D32: renamed from D33; moved to B.Cu
- D33: renamed from D34; moved to B.Cu
- D34: renamed from D35; moved to B.Cu
- D35: renamed from D36; moved to B.Cu
- D36: renamed from D37; moved to B.Cu
- D37: renamed from D38; moved to B.Cu
- D38: renamed from D39; moved to B.Cu
- D39: renamed from D40; moved to B.Cu
- D40: renamed from D41; moved to B.Cu
- D41: renamed from D42; moved to B.Cu
- D42: renamed from D43; moved to B.Cu
- D43: renamed from D44; moved to B.Cu
- D44: renamed from D45; moved to B.Cu
- D45: renamed from D46; moved to B.Cu
- D46: renamed from D47; moved to B.Cu
- D47: renamed from D48; moved to B.Cu
- D48: renamed from D49; moved to B.Cu
- D49: renamed from D50; moved to B.Cu
- D50: renamed from D51; moved to B.Cu
- D51: renamed from D52; moved to B.Cu
- D52: renamed from D53; moved to B.Cu
- D53: renamed from D54; moved to B.Cu
- D54: renamed from D55; moved to B.Cu
- D55: renamed from D56; moved to B.Cu
- D56: renamed from D57; moved to B.Cu
- D57: renamed from D58; moved to B.Cu
- D58: renamed from D59; moved to B.Cu
- D59: renamed from D60; moved to B.Cu
- D60: renamed from D61; moved to B.Cu
- D61: renamed from D62; moved to B.Cu
- D62: renamed from D63; moved to B.Cu
- D63: renamed from D64; moved to B.Cu
- D64: renamed from D65; moved to B.Cu
- D65: renamed from D66; moved to B.Cu
- D66: renamed from D67; moved to B.Cu
- D67: renamed from D68; moved to B.Cu
- D68: renamed from D69; moved to B.Cu
- D69: renamed from D70; moved to B.Cu
- D70: renamed from D71; moved to B.Cu
- D71: renamed from D72; moved to B.Cu
- D72: renamed from D73; moved to B.Cu
- D73: renamed from D74; moved to B.Cu
- D74: renamed from D75; moved to B.Cu
- D75: renamed from D76; moved to B.Cu
- D76: renamed from D77; moved to B.Cu
- D77: renamed from D78; moved to B.Cu
- D78: renamed from D79; moved to B.Cu
- D79: renamed from D80; moved to B.Cu
- D80: renamed from D81; moved to B.Cu
- D81: renamed from D82; moved to B.Cu
- D82: renamed from D83; moved to B.Cu
- D83: renamed from D84; moved to B.Cu
- D84: renamed from D85; moved to B.Cu
- D85: renamed from D86; moved to B.Cu
- D86: renamed from D87; moved to B.Cu
- D87: renamed from D88; moved to B.Cu
- S4: renamed from S5; moved to B.Cu
- S5: renamed from S4; moved to B.Cu
- SW14: renamed from SW15; moved to B.Cu
- SW15: renamed from SW16; moved to B.Cu
- SW16: renamed from SW17; moved to B.Cu
- SW17: renamed from SW18; moved to B.Cu
- SW18: renamed from SW19; moved to B.Cu
- SW19: renamed from SW20; moved to B.Cu
- SW20: renamed from SW21; moved to B.Cu
- SW21: renamed from SW22; moved to B.Cu
- SW22: renamed from SW23; moved to B.Cu
- SW23: renamed from SW24; moved to B.Cu
- SW24: renamed from SW25; moved to B.Cu
- SW25: renamed from SW26; moved to B.Cu
- SW26: renamed from SW27; moved to B.Cu
- SW27: renamed from SW28; moved to B.Cu
- SW28: renamed from SW29; moved to B.Cu
- SW29: renamed from SW30; moved to B.Cu
- SW30: renamed from SW31; moved to B.Cu
- SW31: renamed from SW32; moved to B.Cu
- SW32: renamed from SW33; moved to B.Cu
- SW33: renamed from SW34; moved to B.Cu
- SW34: renamed from SW35; moved to B.Cu
- SW35: renamed from SW36; moved to B.Cu
- SW36: renamed from SW37; moved to B.Cu
- SW37: renamed from SW38; moved to B.Cu
- SW38: renamed from SW39; moved to B.Cu
- SW39: renamed from SW40; moved to B.Cu
- SW40: renamed from SW41; moved to B.Cu
- SW41: renamed from SW42; moved to B.Cu
- SW42: renamed from SW43; moved to B.Cu
- SW43: renamed from SW44; moved to B.Cu
- SW44: renamed from SW45; moved to B.Cu
- SW45: renamed from SW46; moved to B.Cu
- SW46: renamed from SW47; moved to B.Cu
- SW47: renamed from SW48; moved to B.Cu
- SW48: renamed from SW49; moved to B.Cu
- SW49: renamed from SW50; moved to B.Cu
- SW50: renamed from SW51; moved to B.Cu
- SW51: renamed from SW52; moved to B.Cu
- SW52: renamed from SW53; moved to B.Cu
- SW53: renamed from SW54; moved to B.Cu
- SW54: renamed from SW55; moved to B.Cu
- SW55: renamed from SW56; moved to B.Cu
- SW56: renamed from SW57; moved to B.Cu
- SW57: renamed from SW58; moved to B.Cu
- SW58: renamed from SW59; moved to B.Cu
- SW59: renamed from SW60; moved to B.Cu
- SW60: renamed from SW61; moved to B.Cu
- SW61: renamed from SW62; moved to B.Cu
- SW62: renamed from SW63; moved to B.Cu
- SW63: renamed from SW64; moved to B.Cu
- SW64: renamed from SW65; moved to B.Cu
- SW65: renamed from SW66; moved to B.Cu
- SW66: renamed from SW67; moved to B.Cu
- SW67: renamed from SW68; moved to B.Cu
- SW68: renamed from SW69; moved to B.Cu
- SW69: renamed from SW70; moved to B.Cu
- SW70: renamed from SW71; moved to B.Cu
- SW71: renamed from SW72; moved to B.Cu
- SW72: renamed from SW73; moved to B.Cu
- SW73: renamed from SW74; moved to B.Cu
- SW74: renamed from SW75; moved to B.Cu
- SW75: renamed from SW76; moved to B.Cu
- SW76: renamed from SW77; moved to B.Cu
- SW77: renamed from SW78; moved to B.Cu
- SW78: renamed from SW79; moved to B.Cu
- SW79: renamed from SW80; moved to B.Cu
- SW80: renamed from SW81; moved to B.Cu
- SW81: renamed from SW82; moved to B.Cu
- SW82: renamed from SW83; moved to B.Cu
- SW83: renamed from SW84; moved to B.Cu
- SW84: renamed from SW85; moved to B.Cu
- SW85: renamed from SW86; moved to B.Cu
- SW86: renamed from SW87; moved to B.Cu
- SW87: renamed from SW88; moved to B.Cu
- moved F1 361.6 mm to (52.2, 41.7), turned to -90 degrees
- moved C1 311.3 mm to (116.2, 112.0), turned to 180 degrees
- moved U1 311.2 mm to (118.3, 114.3), turned to 180 degrees
- moved C2 304.0 mm to (121.1, 114.3), turned to 90 degrees
- moved C6 283.6 mm to (126.2, 127.8), turned to 180 degrees
- moved C16 267.9 mm to (132.9, 150.4), turned to 135 degrees
- moved R9 267.5 mm to (133.1, 146.8), turned to -135 degrees
- moved R7 267.2 mm to (133.1, 129.1)
- moved R8 264.9 mm to (134.3, 129.1)
- moved Y1 263.9 mm to (134.9, 148.4), turned to 45 degrees
- moved C8 263.9 mm to (129.3, 139.2)
- moved U3 263.9 mm to (134.9, 138.1), turned to 180 degrees
- moved C7 262.9 mm to (129.7, 134.4)
- moved RST1 262.0 mm to (120.7, 144.5), turned to 180 degrees
- moved C15 260.2 mm to (136.8, 150.0), turned to 45 degrees
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Connections:
- R7 pad 1: D+ -> D-
- R8 pad 1: D- -> D+
- U3 pad 23: +3V3 -> +1V1
- U3 pad 43: +1V1 -> +3V3
- U3 pad 45: +3V3 -> +1V1
- U3 pad 48: +1V1 -> +3V3
- U3 pad 50: +3V3 -> +1V1
Routing:
- net D+: track 0.00 -> 180.4 mm
- net D-: track 0.00 -> 179.0 mm
- net +5V: track 0.00 -> 151.1 mm
- net GND: track 0.00 -> 65.3 mm, vias 0 -> 5
- net +3V3: track 0.00 -> 47.4 mm
- net VBUS: track 0.00 -> 14.0 mm
- net +1V1: track 0.00 -> 6.26 mm
- net Net-(U3-USB_DM): track 0.00 -> 5.30 mm
- net Net-(U3-USB_DP): track 0.00 -> 5.27 mm
- net Net-(J2-CC1): track 0.00 -> 3.81 mm
- net Net-(J2-CC2): track 0.00 -> 3.53 mm

Commit message: finished routing mcu and everything besides switch matrix. have to fix usb port
Parts:
- moved C14 5.46 mm to (141.3, 127.5), turned to 180 degrees
- moved R6 4.21 mm to (140.3, 113.8)
- moved R5 3.32 mm to (126.3, 145.9), turned to -90 degrees
- moved R3 2.45 mm to (140.3, 111.1), turned to 180 degrees
- moved C16 1.94 mm to (134.6, 149.4)
- moved R9 1.94 mm to (134.8, 145.9)
- moved Y1 1.94 mm to (136.6, 147.5)
- moved C15 1.94 mm to (138.5, 149.0)
- moved R4 1.76 mm to (140.3, 112.5)
- moved C13 1.49 mm to (134.0, 145.1), turned to -135 degrees
- moved C9 1.37 mm to (141.5, 139.1)
- moved C5 1.30 mm to (135.8, 131.0)
- moved C12 1.30 mm to (134.7, 131.0)
- moved U4 1.19 mm to (147.7, 127.7), turned to 180 degrees
- moved C3 0.76 mm to (133.3, 144.2), turned to -135 degrees
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Connections:
- J3 pad 2: +3V3 -> SWC
- J3 pad 3: GND -> SWD
- J3 pad 4: SWC -> +3V3
- J3 pad 5: SWD -> GND
Routing:
- net +3V3: track 47.4 -> 139.2 mm, vias 0 -> 5
- net Q_SEL: track 0.00 -> 46.1 mm
- net GND: track 65.3 -> 107.4 mm, vias 5 -> 24
- net Q_IO1: track 0.00 -> 23.7 mm
- net RESET: track 0.00 -> 23.5 mm, vias 0 -> 1
- net Q_IO2: track 0.00 -> 22.0 mm
- net +1V1: track 6.26 -> 26.4 mm, vias 0 -> 2
- net SWD: track 0.00 -> 13.9 mm
- net Q_IO3: track 0.00 -> 12.8 mm
- net SWC: track 0.00 -> 12.5 mm
- net Q_CLK: track 0.00 -> 11.7 mm
- net Q_IO0: track 0.00 -> 10.7 mm
- net VBUS: track 14.0 -> 4.96 mm
- net XIN: track 0.00 -> 8.50 mm
- net Net-(BOOT1-Pad2): track 0.00 -> 8.37 mm
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- added copper zone on B.Cu, net GND
- added copper zone on F.Cu, net GND
Other:
- board outline added: 346.1 x 122.2 mm
